File: TempSensingEagleFiles/IOIOShield.brd (EAGLE design)
At the start: 33 x 58.4 mm, 3 parts

Commit message: Revert "STABLE: Added better threading"
This reverts commit b74bb6b943322a5487aef219e170d9d2f1191ec7.
Connections:
- net 3.3V renamed N$5
- net CLK renamed N$6
- net GND renamed N$4
- net SDA renamed N$8
Routing:
- added copper zone on layer 16, net GND
- removed copper zone on layer 16, net N$4
Changed lines of the file:
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@@
 <wire x1="10.74" y1="36.14" x2="10.74" y2="43.48" width="0.8128" layer="16"/>
 </signal>
-<signal name="3.3V">
+<signal name="N$4">
+<contactref element="X4" pad="P$6"/>
+<contactref element="POWER" pad="6"/>
+<wire x1="13.74" y1="21.36" x2="13.74" y2="43.48" width="0.8128" layer="16"/>
+<wire x1="2.54" y1="15.24" x2="7.62" y2="15.24" width="0.8128" layer="16"/>
+<wire x1="7.62" y1="15.24" x2="13.74" y2="21.36" width="0.8128" layer="16"/>
+</signal>
+<signal name="N$5">
 <contactref element="X4" pad="P$7"/>
 <contactref element="POWER" pad="5"/>
@@
 <wire x1="7.62" y1="12.7" x2="16.74" y2="21.82" width="0.8128" layer="16"/>
 </signal>
-<signal name="CLK">
+<signal name="N$6">
 <contactref element="X4" pad="P$4"/>
 <wire x1="22.86" y1="43.36" x2="19.74" y2="46.48" width="0.8128" layer="16"/>
@@
 <wire x1="22.86" y1="20.32" x2="22.86" y2="43.36" width="0.8128" layer="16"/>
 </signal>
-<signal name="SDA">
+<signal name="N$8">
 <contactref element="X4" pad="P$8"/>
 <wire x1="19.74" y1="18.36" x2="19.74" y2="43.48" width="0.8128" layer="16"/>
@@
 <vertex x="-2.54" y="-2.54"/>
 </polygon>
-<contactref element="X4" pad="P$6"/>
-<contactref element="POWER" pad="6"/>
-<wire x1="13.74" y1="21.36" x2="13.74" y2="43.48" width="0.8128" layer="16"/>
-<wire x1="2.54" y1="15.24" x2="7.62" y2="15.24" width="0.8128" layer="16"/>
-<wire x1="7.62" y1="15.24" x2="13.74" y2="21.36" width="0.8128" layer="16"/>
 </signal>
 </signals>

Commit message: STABLE: Added better threading
Connections:
- net N$5 renamed 3.3V
- net N$6 renamed CLK
- net N$8 renamed SDA
- removed net N$4: POWER.6, X4.P$6
- new net GND: POWER.6, X4.P$6
Routing:
- net N$4: track 35.9 -> 0.00 mm
- net GND: track 0.00 -> 35.9 mm
Changed lines of the file:
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@@
 <wire x1="10.74" y1="36.14" x2="10.74" y2="43.48" width="0.8128" layer="16"/>
 </signal>
-<signal name="N$4">
-<contactref element="X4" pad="P$6"/>
-<contactref element="POWER" pad="6"/>
-<wire x1="13.74" y1="21.36" x2="13.74" y2="43.48" width="0.8128" layer="16"/>
-<wire x1="2.54" y1="15.24" x2="7.62" y2="15.24" width="0.8128" layer="16"/>
-<wire x1="7.62" y1="15.24" x2="13.74" y2="21.36" width="0.8128" layer="16"/>
-</signal>
-<signal name="N$5">
+<signal name="3.3V">
 <contactref element="X4" pad="P$7"/>
 <contactref element="POWER" pad="5"/>
@@
 <wire x1="7.62" y1="12.7" x2="16.74" y2="21.82" width="0.8128" layer="16"/>
 </signal>
-<signal name="N$6">
+<signal name="CLK">
 <contactref element="X4" pad="P$4"/>
 <wire x1="22.86" y1="43.36" x2="19.74" y2="46.48" width="0.8128" layer="16"/>
@@
 <wire x1="22.86" y1="20.32" x2="22.86" y2="43.36" width="0.8128" layer="16"/>
 </signal>
-<signal name="N$8">
+<signal name="SDA">
 <contactref element="X4" pad="P$8"/>
 <wire x1="19.74" y1="18.36" x2="19.74" y2="43.48" width="0.8128" layer="16"/>
@@
 <vertex x="-2.54" y="-2.54"/>
 </polygon>
+<contactref element="X4" pad="P$6"/>
+<contactref element="POWER" pad="6"/>
+<wire x1="13.74" y1="21.36" x2="13.74" y2="43.48" width="0.8128" layer="16"/>
+<wire x1="2.54" y1="15.24" x2="7.62" y2="15.24" width="0.8128" layer="16"/>
+<wire x1="7.62" y1="15.24" x2="13.74" y2="21.36" width="0.8128" layer="16"/>
 </signal>
 </signals>
