File: TempSensingEagleFiles/IOIOShield.sch (EAGLE design)
At the start: 3 parts

Commit message: STABLE: Added better threading
Connections:
- net N$4 renamed GND
- net N$5 renamed 3.3V
- net N$6 renamed CLK
- net N$8 renamed SDA
Changed lines of the file:
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@@
 </segment>
 </net>
-<net name="N$4" class="0">
+<net name="GND" class="0">
 <segment>
 <wire x1="38.1" y1="48.26" x2="58.42" y2="48.26" width="0.1524" layer="91"/>
@@
 </segment>
 </net>
-<net name="N$5" class="0">
+<net name="3.3V" class="0">
 <segment>
 <wire x1="38.1" y1="45.72" x2="60.96" y2="45.72" width="0.1524" layer="91"/>
@@
 </segment>
 </net>
-<net name="N$6" class="0">
+<net name="CLK" class="0">
 <segment>
 <pinref part="X4" gate="G$1" pin="4"/>
@@
 </segment>
 </net>
-<net name="N$8" class="0">
+<net name="SDA" class="0">
 <segment>
 <pinref part="X4" gate="G$1" pin="8"/>

Commit message: Revert "STABLE: Added better threading"
This reverts commit b74bb6b943322a5487aef219e170d9d2f1191ec7.
Connections:
- net 3.3V renamed N$5
- net CLK renamed N$6
- net GND renamed N$4
- net SDA renamed N$8
Changed lines of the file:
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@@
 </segment>
 </net>
-<net name="GND" class="0">
+<net name="N$4" class="0">
 <segment>
 <wire x1="38.1" y1="48.26" x2="58.42" y2="48.26" width="0.1524" layer="91"/>
@@
 </segment>
 </net>
-<net name="3.3V" class="0">
+<net name="N$5" class="0">
 <segment>
 <wire x1="38.1" y1="45.72" x2="60.96" y2="45.72" width="0.1524" layer="91"/>
@@
 </segment>
 </net>
-<net name="CLK" class="0">
+<net name="N$6" class="0">
 <segment>
 <pinref part="X4" gate="G$1" pin="4"/>
@@
 </segment>
 </net>
-<net name="SDA" class="0">
+<net name="N$8" class="0">
 <segment>
 <pinref part="X4" gate="G$1" pin="8"/>
